File: keyboard/keyboard-only/keyboard-only.kicad_pcb (KiCad board)
At the start: 2 copper layers, 252.7 x 94 mm, 203 parts, among them J1 USB_C_Receptacle_USB2.0, SW1 SW_PUSH, SW10 SW_PUSH, SW11 SW_PUSH, SW12 SW_PUSH, SW13 SW_PUSH, SW14 SW_PUSH, SW15 SW_PUSH, SW16 SW_PUSH, SW17 SW_PUSH, SW18 SW_PUSH, SW19 SW_PUSH, SW2 SW_PUSH, SW20 SW_PUSH, SW21 SW_PUSH, SW22 SW_PUSH, SW23 SW_PUSH, SW24 SW_PUSH, SW25 SW_PUSH, SW26 SW_PUSH, SW27 SW_PUSH, SW28 SW_PUSH, SW29 SW_PUSH, SW3 SW_PUSH, SW30 SW_PUSH, SW31 SW_PUSH, SW32 SW_PUSH, SW33 SW_PUSH, SW34 SW_PUSH, SW35 SW_PUSH, SW36 SW_PUSH, SW37 SW_PUSH, SW38 SW_PUSH, SW39 SW_PUSH, SW4 SW_PUSH, SW40 SW_PUSH, SW41 SW_PUSH, SW42 SW_PUSH, SW43 SW_PUSH, SW44 SW_PUSH, SW45 SW_PUSH, SW46 SW_PUSH, SW47 SW_PUSH, SW48 SW_PUSH, SW49 SW_PUSH, SW5 SW_PUSH, SW50 SW_PUSH, SW51 SW_PUSH, SW52 SW_PUSH, SW53 SW_PUSH, SW54 SW_PUSH, SW55 SW_PUSH, SW56 SW_PUSH, SW57 SW_PUSH, SW58 SW_PUSH, SW59 SW_PUSH, SW6 SW_PUSH, SW60 SW_PUSH, SW7 SW_PUSH, SW8 SW_PUSH, SW9 SW_PUSH, U1 ATmega16U4-AU, Y1 16MHz

Commit message: Add mounting holes
Parts:
- added Ref**: Val**, kbd:M2_HOLE_v2, F.Cu at (26.0, 97.8)
- added Ref**: Val**, kbd:M2_HOLE_v2, F.Cu at (26.0, 40.6)
- added Ref**: Val**, kbd:M2_HOLE_v2, F.Cu at (270.5, 40.6)
- added Ref**: Val**, kbd:M2_HOLE_v2, F.Cu at (270.5, 97.8)
Routing:
- net COL6: track 236.7 -> 233.7 mm
- net COL8: track 278.8 -> 276.1 mm
- net COL11: track 340.6 -> 337.9 mm
- net COL7: track 257.8 -> 255.1 mm

Commit message: Flip led direction
Parts:
- turned D1 to 90 degrees
- turned D2 to 90 degrees
- turned D3 to 90 degrees
- turned R3 to 90 degrees
- turned R4 to 90 degrees
- turned R5 to 90 degrees
Connections:
- D1 pad 1: N$5 -> GND
- D1 pad 2: GND -> N$4
- D2 pad 1: N$7 -> GND
- D2 pad 2: GND -> N$6
- D3 pad 1: N$3 -> GND
- D3 pad 2: GND -> N$3
- R5 pad 1: VCC -> N$3
- R5 pad 2: N$3 -> VCC
- U1 pad 22: N$6 -> N$7
- U1 pad 8: N$4 -> N$5
Routing:
- net N$7: track 1.93 -> 42.5 mm, vias 0 -> 2
- net N$6: track 42.5 -> 1.93 mm, vias 2 -> 0
- net N$5: track 1.93 -> 32.5 mm, vias 0 -> 2
- net N$4: track 32.5 -> 1.93 mm, vias 2 -> 0
